File: kim-1-RAM-ROM.kicad_pcb (KiCad board)
At the start: 2 copper layers, 113.5 x 134.6 mm, 41 parts, among them J1 Conn_03x06, J2 Conn_03x08, J3 Conn_02x08_Counter_Clockwise, SW1 Image_set, SW2 SW_DIP_x03, SW3 SW_DIP_x07, SW4 SW_DIP_x08, SW5 Vectors, U1 628128, U10 74HCT541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

Commit message: Fix replacing system RAM
Connections:
- U1 pad 24: GND -> /~{R}/W
- U1 pad 29: /R/~{W} -> /RAMR~{W}
- X1 pad V: /R/~{W} -> unconnected-(X1-R/~{W}-PadV)
- X1 pad W: unconnected-(X1-~{R}/W-PadW) -> /~{R}/W
- X1 pad Z: unconnected-(X1-RAMRW-PadZ) -> /RAMR~{W}
Routing:
- net /RAMR~{W}: track 0.00 -> 91.9 mm
- net /~{R}/W: track 0.00 -> 89.8 mm, vias 0 -> 1
- net /R/~{W}: track 83.8 -> 0.00 mm
- net GND: track 101.5 -> 81.4 mm
- net +5V: track 433.1 -> 432.5 mm
